File: Section B - TItle B.kicad_sch (KiCad schematic)
At the start: 0 parts

Commit message: nochmal git add .
Parts:
- added C1: C, symbol Device:C
- added J1: Raspberry_Pi_4, symbol Connector:Raspberry_Pi_4
Connections:
- new net: J1.1 (3V3), J1.17 (3V3)
- new net: C1.1, J1.2 (5V), J1.4 (5V)
- new net GND: C1.2, J1.14 (GND), J1.20 (GND), J1.25 (GND), J1.30 (GND), J1.34 (GND), J1.39 (GND), J1.6 (GND), J1.9 (GND)
